File: pcb/_autosave-flight_comp_srad-2026.kicad_sch (KiCad schematic)
At the start: 61 parts, among them J1 503398-1892, J3 USB_B_Micro, U1 IIM-20670, U2 NCP1117-3.3_SOT223, U3 RP2040, U4 ADXL375BCCZ-RL7, U5 MAX-M10M-00B, U6 W25Q128JVS, U7 XBP9B-DMSTB002, Y1 ABM8-272-T3

Commit message: updated datasheets for xbee
Other:
- note added: "XBEE Pro SX 900 RF RF transceiver"
- note removed: "XBEE SX900RF RF transceiver"
Changed lines of the file:
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@@
 		)
 	)
-	(text "XBEE SX900RF\nRF transceiver"
+	(text "XBEE Pro SX 900 RF\nRF transceiver"
 		(exclude_from_sim no)
 		(at 228.854 303.53 0)
