File: pcb/_autosave-flight_comp_srad-2026.kicad_sch (KiCad schematic)
At the start: 69 parts, among them J1 503398-1892, J2 Connector_3, J3 USB_B_Micro, J5 Vin_Bat, U1 IIM-20670, U2 NCP1117-3.3_SOT223, U3 RP2040, U4 ADXL375BCCZ-RL7, U5 MAX-M10M-00B, U6 W25Q128JVS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

Commit message: Cambio de regulador de tensión - chequear impedancia de línea
Parts:
- added U8: TPS73733DCQ, Package_TO_SOT_SMD:SOT-223-6, symbol TPS73733DCQ:TPS73733DCQ
Connections:
- net +3V3: now also U8.2 (OUT); no longer U2.2 (VO)
- net GND: now also U8.3 (GND-1), U8.6 (GND)
- net VBUS: now also U8.1 (IN), U8.5 (EN); no longer U2.3 (VI)
- no-connect marks 33 -> 34
Other:
- note removed: "chequear la impedancia de la linea del USB"
- moved on the sheet: CFLASH_1, CPS_1, CPS_2, CX_1, CX_2, Div_res_bat1, Div_res_bat2, J5, RFLASH_1, RFLASH_2, RX_1, S1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
