File: pcb/_autosave-flight_comp_srad-2026.kicad_sch (KiCad schematic)
At the start: 75 parts, among them J1 503398-1892, J2 Connector_3, J3 USB_B_Micro, J5 Vin_Bat, U1 IIM-20670, U3 RP2040, U4 ADXL375BCCZ-RL7, U5 MAX-M10M-00B, U6 W25Q128JVS, U7 XBP9B-DMSTB002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

Commit message: quedan 62 errores de DRC mas warnings
principales errores:
- clearance violation (no sé por qué está en 0.2mm pero no puedo cambiarlo XD)
- cortos por las vias más grandes
- boludeces de la serigrafía, habría que volar todo lo que no sea importante
- falta poner shunt a la linea de tx, no se como porque no entra XD
- más boludeces como la posición del USB, está bien que sobresalga (ver capa user drawings) pero da error
Other:
- note added: "JLC04161H-7628E W=0.7 Gap=0.4 Thickness=0.4284 mm"
- note removed: "JLC04161H-7628C W=0.9 Gap=0.3 Thickness=0.646 mm"
Changed lines of the file:
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@@
 		)
 	)
-	(text "JLC04161H-7628C\nW=0.9\nGap=0.3\nThickness=0.646 mm"
+	(text "JLC04161H-7628E\nW=0.7\nGap=0.4\nThickness=0.4284 mm"
 		(exclude_from_sim no)
 		(at 132.334 145.542 0)
