File: pcb/flight_comp_srad-2026.kicad_sch (KiCad schematic)
At the start: 61 parts, among them J1 503398-1892, J3 USB_B_Micro, U1 IIM-20670, U2 NCP1117-3.3_SOT223, U3 RP2040, U4 ADXL375BCCZ-RL7, U5 MAX-M10M-00B, U6 W25Q128JVS, U7 XBP9B-DMSTB002, Y1 ABM8-272-T3

Commit message: cosas del xbee
Parts:
- added CXB_1, CXB_2: C, TCLib:C_0805, symbol TCLib:C
- U7: footprint RF_Module:Digi_XBee_SMT -> SRAD_fligh_comp2026:XBEEPRO
Connections:
- net +3V3: now also CXB_1.1, CXB_2.1
- net GND: now also CXB_1.2, CXB_2.2
Other:
- note added: "Closest -> Furthest"
- note added: "XBEE Pro SX 900 RF RF transceiver"
- note removed: "XBEE SX900RF RF transceiver"

Commit message: footprints y cosas
Parts:
- CXB_1: value C -> 47p
- CXB_2: value C -> 1u
Connections:
- net +3V3: no longer U5.6 (V_BCKP)
- net GND: now also U7.14 (VREF)
- no-connect marks 13 -> 28
Other:
- note added: "XBEE Pro S3B 900HP RF transceiver"
- note added: "chequear footprint!!!!!!! me fije y esta bien para mi -Vito"
- note removed: "XBEE Pro SX 900 RF RF transceiver"
- note removed: "chequear footprint!!!!!!!"
- moved on the sheet: CXB_2
Changed lines of the file:
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@@
 		)
 	)
-	(text "XBEE Pro SX 900 RF\nRF transceiver"
+	(text "XBEE Pro S3B 900HP\nRF transceiver"
 		(exclude_from_sim no)
 		(at 228.854 303.53 0)
@@
 	(text "Cap 1u tantalio"
 		(exclude_from_sim no)
-		(at 91.694 247.904 0)
+		(at 48.768 250.952 0)
 		(effects
 			(font
@@
 		)
 	)
-	(text "chequear footprint!!!!!!!"
+	(text "chequear footprint!!!!!!!\n\nme fije y esta bien para mi\n-Vito"
 		(exclude_from_sim no)
-		(at 115.57 310.896 0)
+		(at 121.412 366.776 0)
 		(effects
 			(font
@@
 	)
 	(junction
-		(at 269.24 328.93)
+		(at 271.78 328.93)
 		(diameter 0)
 		(color 0 0 0 0)
@@
 	)
 	(junction
-		(at 102.87 127)
-		(diameter 0)
-		(color 0 0 0 0)
-	)
-	(junction
 		(at 389.89 232.41)
 		(diameter 0)
@@
 	)
 	(no_connect
+		(at 199.39 351.79)
+	)
+	(no_connect
 		(at 100.33 147.32)
 	)
@@
 	)
 	(no_connect
+		(at 199.39 328.93)
+	)
+	(no_connect
 		(at 219.71 234.95)
 	)
 	(no_connect
+		(at 199.39 349.25)
+	)
+	(no_connect
 		(at 55.88 228.6)
 	)
@@
 	)
 	(no_connect
+		(at 255.27 356.87)
+	)
+	(no_connect
+		(at 199.39 344.17)
+	)
+	(no_connect
+		(at 199.39 369.57)
+	)
+	(no_connect
+		(at 199.39 364.49)
+	)
+	(no_connect
 		(at 54.61 134.62)
 	)
 	(no_connect
+		(at 199.39 359.41)
+	)
+	(no_connect
+		(at 199.39 356.87)
+	)
+	(no_connect
+		(at 199.39 367.03)
+	)
+	(no_connect
+		(at 199.39 331.47)
+	)
+	(no_connect
 		(at 54.61 149.86)
 	)
+	(no_connect
+		(at 100.33 129.54)
+	)
+	(no_connect
+		(at 199.39 354.33)
+	)
+	(no_connect
+		(at 199.39 346.71)
+	)
+	(no_connect
+		(at 199.39 361.95)
+	)
 	(wire
 		(pts
@@
 	(wire
 		(pts
-			(xy 102.87 127) (xy 102.87 129.54)
-		)
-		(stroke
-			(width 0)
-			(type default)
-		)
-	)
-	(wire
-		(pts
 			(xy 473.71 30.48) (xy 485.14 30.48)
 		)
@@
 	(wire
 		(pts
-			(xy 259.08 340.36) (xy 269.24 340.36)
+			(xy 259.08 340.36) (xy 271.78 340.36)
 		)
 		(stroke
@@
 	(wire
 		(pts
-			(xy 269.24 330.2) (xy 269.24 328.93)
+			(xy 271.78 330.2) (xy 271.78 328.93)
 		)
 		(stroke
@@
 	(wire
 		(pts
-			(xy 269.24 325.12) (xy 269.24 328.93)
+			(xy 271.78 325.12) (xy 271.78 328.93)
 		)
 		(stroke
@@
 	(wire
 		(pts
-			(xy 102.87 129.54) (xy 100.33 129.54)
-		)
-		(stroke
-			(width 0)
-			(type default)
-		)
-	)
-	(wire
-		(pts
 			(xy 419.1 46.99) (xy 419.1 45.72)
 		)
@@
 	(wire
 		(pts
+			(xy 199.39 334.01) (xy 190.5 334.01)
+		)
+		(stroke
+			(width 0)
+			(type default)
+		)
+	)
+	(wire
+		(pts
 			(xy 177.8 237.49) (xy 177.8 240.03)
 		)
@@
 	(wire
 		(pts
-			(xy 259.08 328.93) (xy 269.24 328.93)
+			(xy 259.08 328.93) (xy 271.78 328.93)
 		)
 		(stroke
@@
 	(wire
 		(pts
-			(xy 269.24 340.36) (xy 269.24 337.82)
+			(xy 271.78 340.36) (xy 271.78 337.82)
 		)
 		(stroke
@@
 	(wire
 		(pts
+			(xy 190.5 331.47) (xy 190.5 334.01)
+		)
+		(stroke
+			(width 0)
+			(type default)
+		)
+	)
+	(wire
+		(pts
 			(xy 447.04 50.8) (xy 449.58 50.8)
 		)
@@
 	(symbol
 		(lib_id "power:+3V3")
-		(at 269.24 325.12 0)
+		(at 271.78 325.12 0)
 		(unit 1)
 		(exclude_from_sim no)
@@
 		(fields_autoplaced yes)
 		(property "Reference" "#PWR03"
-			(at 269.24 328.93 0)
+			(at 271.78 328.93 0)
 			(effects
 				(font
@@
 		)
 		(property "Value" "+3V3"
-			(at 269.24 320.04 0)
+			(at 271.78 320.04 0)
 			(effects
 				(font
@@
 		)
 		(property "Footprint" ""
-			(at 269.24 325.12 0)
+			(at 271.78 325.12 0)
 			(effects
 				(font
@@
 		)
 		(property "Datasheet" ""
-			(at 269.24 325.12 0)
+			(at 271.78 325.12 0)
 			(effects
 				(font
@@
 		)
 		(property "Description" "Power symbol creates a global label with name \"+3V3\""
-			(at 269.24 325.12 0)
+			(at 271.78 325.12 0)
 			(effects
 				(font
@@
 	)
 	(symbol
+		(lib_id "power:GND")
+		(at 190.5 331.47 180)
+		(unit 1)
+		(exclude_from_sim no)
+		(in_bom yes)
+		(on_board yes)
+		(dnp no)
+		(fields_autoplaced yes)
+		(property "Reference" "#PWR057"
+			(at 190.5 325.12 0)
+			(effects
+				(font
+					(size 1.27 1.27)
+				)
+				(hide yes)
+			)
+		)
+		(property "Value" "GND"
+			(at 190.5 326.39 0)
+			(effects
+				(font
+					(size 1.27 1.27)
+				)
+			)
+		)
+		(property "Footprint" ""
+			(at 190.5 331.47 0)
+			(effects
+				(font
+					(size 1.27 1.27)
+				)
+				(hide yes)
+			)
+		)
+		(property "Datasheet" ""
+			(at 190.5 331.47 0)
+			(effects
+				(font
+					(size 1.27 1.27)
+				)
+				(hide yes)
+			)
+		)
+		(property "Description" "Power symbol creates a global label with name \"GND\" , ground"
+			(at 190.5 331.47 0)
+			(effects
+				(font
+					(size 1.27 1.27)
+				)
+				(hide yes)
+			)
+		)
+		(pin "1"
+		)
+		(instances
+			(project ""
+				(path "/142d7a80-3dfb-4605-bdd8-7dd9e7ca17c7"
+					(reference "#PWR057")
+					(unit 1)
+				)
+			)
+		)
+	)
+	(symbol
 		(lib_name "GND_8")
 		(lib_id "power:GND")
@@
 			)
 		)
-		(property "Value" "C"
+		(property "Value" "47p"
 			(at 262.89 335.2799 0)
 			(effects
@@
 	(symbol
 		(lib_id "TCLib:C")
-		(at 269.24 334.01 0)
+		(at 271.78 334.01 0)
 		(unit 1)
 		(exclude_from_sim no)
@@
 		(fields_autoplaced yes)
 		(property "Reference" "CXB_2"
-			(at 273.05 332.7399 0)
+			(at 275.59 332.7399 0)
 			(effects
 				(font
@@
 			)
 		)
-		(property "Value" "C"
-			(at 273.05 335.2799 0)
+		(property "Value" "1u"
+			(at 275.59 335.2799 0)
 			(effects
 				(font
@@
 		)
 		(property "Footprint" "TCLib:C_0805"
-			(at 252.73 330.708 0)
+			(at 255.27 330.708 0)
 			(effects
 				(font
@@
 		)
 		(property "Datasheet" "~"
-			(at 269.24 334.01 0)
+			(at 271.78 334.01 0)
 			(effects
 				(font
@@
 		)
 		(property "Description" "Unpolarized capacitor"
-			(at 251.968 326.136 0)
+			(at 254.508 326.136 0)
 			(effects
 				(font

Commit message: queda cablear los gpios
Parts:
- added J2: Connector_3, TCLib:PinHeader_1x03_P2.54mm_Vertical, symbol TCLib:Connector_3
- added JP1: SolderJumper_2_Open, Jumper:SolderJumper-2_P1.3mm_Open_TrianglePad1.0x1.5mm, symbol Jumper:SolderJumper_2_Open
- added R_RST1: 10k, Resistor_SMD:R_0402_1005Metric, symbol Device:R
- added S2: PTS810SJK250SMTR_LFS, SRAD_fligh_comp2026:PTS810SJK250SMTRLFS, symbol SRAD:PTS810SJK250SMTR_LFS
- S1: footprint PTS810SJK250SMTRLFS:PTS810SJK250SMTRLFS -> SRAD_fligh_comp2026:PTS810SJK250SMTRLFS
Connections:
- net +3V3: now also R_RST1.1
- net GND: now also J2.1, S2.3 (COM_1), S2.4 (COM_2)
- net at U3.2 (GPIO0): now also JP1.1 (A)
- net SWCLK: now reaches U3.24 (SWCLK)
- net SWCLK: now also J2.3
- net SWDIO: now reaches U3.25 (SWD)
- net SWDIO: now also J2.2
- net RUN: now reaches U3.26 (RUN)
- net RUN: now also R_RST1.2, S2.1 (NO_1), S2.2 (NO_2)
- net PPS: now reaches U5.4 (TIMEPULSE)
- net PPS: now also JP1.2 (B)
- no-connect marks 28 -> 29
Other:
- note added: "Debug Interface"
- note added: "Reset Button"
- moved on the sheet: A1, AE1, C10, C11, C12, C13, C14, C15, C16, C17, C6, C7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

Commit message: plano de masa y antena puestos
Parts:
- CADXL_1: footprint Capacitor_SMD:C_0805_2012Metric -> Capacitor_SMD:C_0402_1005Metric
- CXB_1, CXB_2: footprint TCLib:C_0805 -> Capacitor_SMD:C_0603_1608Metric
Changed lines of the file:
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@@
 			)
 		)
-		(property "Footprint" "Capacitor_SMD:C_0805_2012Metric"
+		(property "Footprint" "Capacitor_SMD:C_0402_1005Metric"
 			(at 53.0352 260.35 0)
 			(effects
@@
 			)
 		)
-		(property "Footprint" "TCLib:C_0805"
+		(property "Footprint" "Capacitor_SMD:C_0603_1608Metric"
 			(at 233.68 330.708 0)
 			(effects
@@
 			)
 		)
-		(property "Footprint" "TCLib:C_0805"
+		(property "Footprint" "Capacitor_SMD:C_0603_1608Metric"
 			(at 246.38 330.708 0)
 			(effects

Commit message: conectado spi del iim y ruteo de algunos caps de desacople
Parts:
- removed JP1: SolderJumper_2_Open, Jumper:SolderJumper-2_P1.3mm_Open_TrianglePad1.0x1.5mm, symbol Jumper:SolderJumper_2_Open
- added RI2C_3, RI2C_4: 10k, Resistor_SMD:R_0402_1005Metric, symbol Device:R
Connections:
- net IIM_CS is gone; now on net IIM_CS1: U1.23 (NCS)
- net IIM_MISO is gone; now on net IIM_MISO1: U1.9 (MISO)
- net IIM_MOSI is gone; now on net IIM_MOSI1: U1.1 (MOSI)
- net IIM_SCLK is gone; now on net IIM_SCLK1: U1.24 (SCLK)
- net UART_Rx is gone; now on net UART_Rx0: U7.2 (DOUT/DIO13)
- net UART_Tx is gone; now on net UART_Tx0: U7.3 (DIN/NCONFIG/DIO14)
- net +3V3: now also RI2C_3.2, RI2C_4.2
- net ADXL_SCL: now also U3.5 (GPIO3); no longer U3.7 (GPIO5), U5.17 (SCL)
- net ADXL_SDA: now also U3.4 (GPIO2); no longer U3.6 (GPIO4), U5.16 (SDA)
- net IIM_MISO1: now reaches U3.11 (GPIO8)
- net IIM_CS1: now reaches U3.12 (GPIO9)
- net IIM_SCLK1: now reaches U3.13 (GPIO10)
- net IIM_MOSI1: now reaches U3.14 (GPIO11)
- net UART_Tx0: now reaches U3.2 (GPIO0)
- net UART_Rx0: now reaches U3.3 (GPIO1)
- net PPS: no longer names the net of U5.4 (TIMEPULSE)
- new net GNSS_SCL: RI2C_3.1, U3.7 (GPIO5), U5.17 (SCL)
- new net GNSS_SDA: RI2C_4.1, U3.6 (GPIO4), U5.16 (SDA)
- no-connect marks 29 -> 30
Other:
- note added: "I2C0 bus"
- note added: "I2C1 bus"
- note removed: "I2C port"
- note removed: "chequear footprint!!!!!!! me fije y esta bien para mi -Vito"
- moved on the sheet: A1, C10, C11, C12, C13, C14, C15, C16, C17, C6, C7, C8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

Commit message: listo los caps de desacople de la rp2040
Parts:
- C10, C11, C12, C13, C14, C15, C16, C17, C6, C7, C8, C9: footprint Capacitor_SMD:C_0805_2012Metric -> Capacitor_SMD:C_0402_1005Metric
Other:
- note added: "falta poner botones"
- moved on the sheet: J2, RI2C_1, RI2C_2, RI2C_3, RI2C_4, R_RST1, S2

Commit message: listo el routeo de casi todo falta layer gnd y 3v3, capas adxl
Parts:
- CBAR_1, CBAR_2, CFLASH_1, CGPS_1, CGPS_2, CGPS_3, CIIM_1, CIIM_2, CIIM_3, CIIM_4: footprint Capacitor_SMD:C_0805_2012Metric -> Capacitor_SMD:C_0402_1005Metric
Connections:
- net UART_Rx0: now also U3.28 (GPIO17); no longer U3.3 (GPIO1)
- net UART_Tx0: now also U3.27 (GPIO16); no longer U3.2 (GPIO0)
- net RP_SDA0: now reaches U3.15 (GPIO12)
- net RP_SDA0: now also RI2C_4.1, U5.16 (SDA)
- net RP_SCL0: now reaches U3.16 (GPIO13)
- net RP_SCL0: now also RI2C_3.1, U5.17 (SCL)
- net ADXL_SCL renamed RP_SCL1
- net ADXL_SDA renamed RP_SDA1
- removed net GNSS_SCL: RI2C_3.1, U3.7 (GPIO5), U5.17 (SCL)
- removed net GNSS_SDA: RI2C_4.1, U3.6 (GPIO4), U5.16 (SDA)
Other:
- note added: "GNSS"
- note added: "Has to be close to a mounting hole for stability"
- note added: "MS5611 & ADXL"
- note added: "chequear footprint cap tantalio"
- note added: "no se si hace falta ese cap de desacople"
- note added: "usamos interrupciones para el ADXL?"
- moved on the sheet: RI2C_1, RI2C_2, RI2C_3, RI2C_4

Commit message: Planos de 3V3 y VBUS, y otras cositas
Planos de 3V3 y VBUS, y otras cositas
Parts:
- added J5: Vin_Bat, TCLib:Molex_1x02_P2.54mm, symbol TCLib:Connector_2_Pol
Connections:
- net GND: now also J5.2
- net VBUS: now also J5.1
- no-connect marks 30 -> 32
Other:
- moved on the sheet: CPS_1, CPS_2, J3, U2
