File: pcb/flight_comp_srad-2026.kicad_sch (KiCad schematic)
At the start: 70 parts, among them J1 503398-1892, J2 Connector_3, J3 USB_B_Micro, J5 Vin_Bat, U1 IIM-20670, U2 NCP1117-3.3_SOT223, U3 RP2040, U4 ADXL375BCCZ-RL7, U5 MAX-M10M-00B, U6 W25Q128JVS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

Commit message: Realimentación bien hecha y agujeros ajustados
Parts:
- removed U2: NCP1117-3.3_SOT223, Package_TO_SOT_SMD:SOT-223-3_TabPin2, symbol Regulator_Linear:NCP1117-3.3_SOT223
- added CPS_3: 10u, Capacitor_SMD:C_0805_2012Metric, symbol Device:C
- added Div_res_reg1a1, Div_res_reg2a1: 82k, Resistor_SMD:R_0805_2012Metric, symbol Device:R
- added Div_res_reg1b1: 150k, Resistor_SMD:R_0805_2012Metric, symbol Device:R
- added Div_res_reg2b1: 47k, Resistor_SMD:R_0805_2012Metric, symbol Device:R
- Div_res_bat1, Div_res_bat2, RL_1, RL_2: footprint Resistor_SMD:R_0402_1005Metric -> Resistor_SMD:R_0805_2012Metric
Connections:
- net +3V3: now also CPS_3.1, Div_res_reg1a1.2, Div_res_reg1b1.2
- net GND: now also Div_res_reg2a1.2, Div_res_reg2b1.2
- net NR_Reg: now reaches U8.4 (NR/FB)
- net NR_Reg: now also CPS_3.2, Div_res_reg1a1.1, Div_res_reg1b1.1, Div_res_reg2a1.1, Div_res_reg2b1.1
- no-connect marks 34 -> 33
Other:
- moved on the sheet: CFLASH_1, CPS_1, CPS_2, CX_1, CX_2, Div_res_bat1, Div_res_bat2, J3, J5, RFLASH_1, RFLASH_2, RX_1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

Commit message: Final?
Can you beat KiCAD with dementia?
Parts:
- CX_1, CX_2: footprint Capacitor_SMD:C_0201_0603Metric -> Capacitor_SMD:C_0805_2012Metric
- RX_1: footprint Resistor_SMD:R_0201_0603Metric -> Resistor_SMD:R_0805_2012Metric
- R_RST1: footprint Resistor_SMD:R_0402_1005Metric -> Resistor_SMD:R_0805_2012Metric
Changed lines of the file:
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@@
 			)
 		)
-		(property "Footprint" "Resistor_SMD:R_0201_0603Metric"
+		(property "Footprint" "Resistor_SMD:R_0805_2012Metric"
 			(at 363.22 64.008 90)
 			(effects
@@
 			)
 		)
-		(property "Footprint" "Resistor_SMD:R_0402_1005Metric"
+		(property "Footprint" "Resistor_SMD:R_0805_2012Metric"
 			(at 310.642 220.98 90)
 			(effects
@@
 			)
 		)
-		(property "Footprint" "Capacitor_SMD:C_0201_0603Metric"
+		(property "Footprint" "Capacitor_SMD:C_0805_2012Metric"
 			(at 334.518 78.74 0)
 			(effects
@@
 			)
 		)
-		(property "Footprint" "Capacitor_SMD:C_0201_0603Metric"
+		(property "Footprint" "Capacitor_SMD:C_0805_2012Metric"
 			(at 334.518 52.07 0)
 			(effects

Commit message: cambio P-UPs y BOOT a 0805
Parts:
- RFLASH_1, RFLASH_2, RI2C_3, RI2C_4: footprint Resistor_SMD:R_0402_1005Metric -> Resistor_SMD:R_0805_2012Metric
Changed lines of the file:
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@@
 			)
 		)
-		(property "Footprint" "Resistor_SMD:R_0402_1005Metric"
+		(property "Footprint" "Resistor_SMD:R_0805_2012Metric"
 			(at 252.222 48.26 90)
 			(effects
@@
 			)
 		)
-		(property "Footprint" "Resistor_SMD:R_0402_1005Metric"
+		(property "Footprint" "Resistor_SMD:R_0805_2012Metric"
 			(at 183.388 208.28 90)
 			(effects
@@
 			)
 		)
-		(property "Footprint" "Resistor_SMD:R_0402_1005Metric"
+		(property "Footprint" "Resistor_SMD:R_0805_2012Metric"
 			(at 227.838 208.28 90)
 			(effects
@@
 			)
 		)
-		(property "Footprint" "Resistor_SMD:R_0402_1005Metric"
+		(property "Footprint" "Resistor_SMD:R_0805_2012Metric"
 			(at 245.11 52.832 90)
 			(effects

Commit message: agregue beeper que falta conectar, saque vias abajo de pads y saque la filling zone gnd del bottom del regulador
Parts:
- added LS1: PS1240P02BT, Buzzer_Beeper:Buzzer_TDK_PS1240P02BT_D12.2mm_H6.5mm, symbol PS1240P02BT:PS1240P02BT
Connections:
- net GND: now also LS1.2
- net BUZZER: now reaches U3.2 (GPIO0)
- net BUZZER: now also LS1.1

Commit message: beeper listo
Parts:
- added Q1: BC547, Package_TO_SOT_THT:TO-92_Inline, symbol Transistor_BJT:BC547
- added R1: R, Resistor_SMD:R_0805_2012Metric, symbol Device:R
- added R2: 1k, Resistor_SMD:R_0805_2012Metric, symbol Device:R
Connections:
- net BUZZER: now also R1.1; no longer LS1.1
- net GND: now also Q1.3 (E); no longer LS1.2
- new net: Q1.2 (B), R1.2
- new net: LS1.2, Q1.1 (C), R2.1
- new net 3V3: LS1.1, R2.2
Other:
- moved on the sheet: LS1

Commit message: beeper listo listo
Connections:
- net 3V3 is gone; now on net +3V3: LS1.1, R2.2
Changed lines of the file:
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@@
 	)
 	(junction
-		(at 537.21 255.27)
-		(diameter 0)
-		(color 0 0 0 0)
-	)
-	(junction
 		(at 90.17 369.57)
 		(diameter 0)
@@
 	)
 	(junction
+		(at 537.21 255.27)
+		(diameter 0)
+		(color 0 0 0 0)
+	)
+	(junction
 		(at 121.92 50.8)
 		(diameter 0)
@@
 	(wire
 		(pts
+			(xy 537.21 252.73) (xy 537.21 255.27)
+		)
+		(stroke
+			(width 0)
+			(type default)
+		)
+	)
+	(wire
+		(pts
 			(xy 547.37 269.24) (xy 537.21 269.24)
 		)
@@
 	(wire
 		(pts
-			(xy 537.21 252.73) (xy 537.21 255.27)
-		)
-		(stroke
-			(width 0)
-			(type default)
-		)
-	)
-	(wire
-		(pts
 			(xy 90.17 364.49) (xy 90.17 367.03)
 		)
@@
 		)
 	)
-	(label "3V3"
-		(at 537.21 252.73 0)
-		(effects
-			(font
-				(size 1.27 1.27)
-			)
-			(justify left bottom)
-		)
-	)
 	(label "~{USB_BOOT}"
 		(at 229.87 54.61 0)
@@
 					(unit 1)
 				)
+			)
+		)
+	)
+	(symbol
+		(lib_id "power:+3V3")
+		(at 537.21 252.73 0)
+		(unit 1)
+		(exclude_from_sim no)
+		(in_bom yes)
+		(on_board yes)
+		(dnp no)
+		(fields_autoplaced yes)
+		(property "Reference" "#PWR034"
+			(at 537.21 256.54 0)
+			(effects
+				(font
+					(size 1.27 1.27)
+				)
+				(hide yes)
+			)
+		)
+		(property "Value" "+3V3"
+			(at 537.21 247.65 0)
+			(effects
+				(font
+					(size 1.27 1.27)
+				)
+			)
+		)
+		(property "Footprint" ""
+			(at 537.21 252.73 0)
+			(effects
+				(font
+					(size 1.27 1.27)
+				)
+				(hide yes)
+			)
+		)
+		(property "Datasheet" ""
+			(at 537.21 252.73 0)
+			(effects
+				(font
+					(size 1.27 1.27)
+				)
+				(hide yes)
+			)
+		)
+		(property "Description" "Power symbol creates a global label with name \"+3V3\""
+			(at 537.21 252.73 0)
+			(effects
+				(font
+					(size 1.27 1.27)
+				)
+				(hide yes)
+			)
+		)
+		(pin "1"
+		)
+		(instances
+			(project ""
+				(path "/142d7a80-3dfb-4605-bdd8-7dd9e7ca17c7"
+					(reference "#PWR034")
+					(unit 1)
+				)
