File: pcb/flight_comp_srad-2026.kicad_pcb (KiCad board)
At the start: 4 copper layers, 70 x 40 mm, 65 parts, among them J1 503398-1892, J2 Connector_3, J3 USB_B_Micro, J5 Vin_Bat, U1 IIM-20670, U2 NCP1117-3.3_SOT223, U3 RP2040, U4 ADXL375BCCZ-RL7, U5 MAX-M10M-00B, U6 W25Q128JVS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

Commit message: Pistas terminadas (FALTA REVISAR) + medidor tensión batería
Parts:
- added Div_res_bat1: 100k, Resistor_SMD:R_0402_1005Metric, F.Cu at (203.8, 94.6)
- added Div_res_bat2: 470k, Resistor_SMD:R_0402_1005Metric, F.Cu at (203.0, 92.8)
- moved CIIM_4 8.57 mm to (190.8, 76.4), turned to -90 degrees
- moved CADXL_2 6.65 mm to (213.0, 65.0)
- moved CIIM_3 5.78 mm to (190.2, 73.4)
- moved CADXL_1 5.58 mm to (204.0, 64.6), turned to 90 degrees
- moved CBAR_2 5.20 mm to (203.2, 77.6)
- moved CIIM_2 5.00 mm to (198.4, 74.4), turned to -90 degrees
- moved D1 1.97 mm to (200.2, 96.4)
- moved D2 1.97 mm to (202.2, 96.4)
- moved RL_1 1.60 mm to (200.2, 99.2)
- moved RL_2 1.60 mm to (202.2, 99.2)
- moved CBAR_1 1.00 mm to (200.2, 71.8), turned to 90 degrees
- moved CIIM_1 0.19 mm to (190.2, 74.6)
Connections:
- U3 pad 40: unconnected-(U3-GPIO28_ADC2-Pad40) -> /ADC_BAT
Routing:
- net GND: track 67.7 -> 116.9 mm, vias 28 -> 35
- net +3V3: track 103.6 -> 151.8 mm, vias 24 -> 32
- net VBUS: track 5.98 -> 19.9 mm, vias 1 -> 2
- net /ADC_BAT: track 0.00 -> 5.69 mm
- net Net-(D2-K): track 2.10 -> 0.00 mm
- net /IIM_MISO1: track 16.2 -> 18.2 mm
- net /RP_SDA1: track 21.1 -> 22.6 mm
- net /LED_1: track 5.15 -> 6.66 mm
- net /LED_2: track 5.81 -> 6.62 mm
- net Net-(D1-K): track 2.10 -> 1.49 mm

Commit message: Pistas terminadas (FALTA REVISAR) + medidor tensión batería
Me faltó poner una pista más xd
Routing:
- net Net-(D2-K): track 0.00 -> 1.49 mm
Changed lines of the file:
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@@
 		(net 92)
+	)
+	(segment
+		(start 202.2 98.665)
+		(end 202.2 97.175)
+		(width 0.2)
+		(layer "F.Cu")
+		(net 93)
 	)
 	(zone

Commit message: routeo listo, falta revisar las conecc
Parts:
- added G***: LOGO, my_lib:Logo_ITBA_rocketry, F.Cu at (197.6, 69.0)
- added S2: PTS810SJK250SMTR_LFS, SRAD_fligh_comp2026:PTS810SJK250SMTRLFS, F.Cu at (193.2, 93.0)
- moved J2 0.70 mm to (192.0, 98.7)
Routing:
- net GND: track 116.9 -> 128.2 mm
- net /RUN: track 4.21 -> 12.9 mm
- net /SD_DAT0: track 27.5 -> 28.5 mm
- net /SWDIO: track 12.5 -> 13.3 mm
- net /SWCLK: track 12.5 -> 13.2 mm

Commit message: agregue coments
Changed lines of the file:
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@@
 	)
 	(segment
-		(start 190.699 88.099)
-		(end 190.8 88.2)
+		(start 190.301 88.2)
+		(end 191.49 88.2)
 		(width 0.2)
 		(layer "F.Cu")
@@
 		(start 212.835 68.05)
 		(end 212.835 67.16)
-		(width 0.2)
-		(layer "F.Cu")
-		(net 47)
-	)
-	(segment
-		(start 190.8 88.2)
-		(end 191.49 88.2)
 		(width 0.2)
 		(layer "F.Cu")
@@
 	)
 	(segment
-		(start 190.2 88.099)
-		(end 190.699 88.099)
-		(width 0.2)
-		(layer "F.Cu")
-		(net 47)
-	)
-	(segment
 		(start 204.5 88.708521)
 		(end 204.5 88.9)
 		(width 0.2)
 		(layer "F.Cu")
+		(net 47)
+	)
+	(segment
+		(start 190.2 88.099)
+		(end 190.301 88.2)
+		(width 0.2)
+		(layer "F.Cu")

Commit message: Cambio plano 3v3
Routing:
- net +3V3: track 151.8 -> 145.4 mm
Changed lines of the file:
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@@
 	)
 	(segment
-		(start 183.125 62.475)
-		(end 184.05 62.475)
-		(width 0.5)
+		(start 182.25 63.85)
+		(end 183.549 62.551)
+		(width 1)
 		(layer "F.Cu")
 		(net 6)
 	)
 	(segment
-		(start 182.25 63.35)
-		(end 183.125 62.475)
-		(width 0.5)
+		(start 183.549 62.551)
+		(end 184.05 62.551)
+		(width 1)
 		(layer "F.Cu")
 		(net 6)
@@
 	(segment
 		(start 182.25 69.2875)
-		(end 182.25 63.35)
-		(width 0.5)
+		(end 182.25 63.85)
+		(width 1)
 		(layer "F.Cu")
 		(net 6)
@@
 	)
 	(segment
-		(start 212.825 68.375)
-		(end 209.2 72)
-		(width 0.4)
-		(layer "In2.Cu")
-		(net 47)
-	)
-	(segment
 		(start 181.8 100)
 		(end 181.8 94)
@@
 	)
 	(segment
-		(start 212.825 67.15)
-		(end 212.825 68.375)
-		(width 0.4)
-		(layer "In2.Cu")
-		(net 47)
-	)
-	(segment
 		(start 195.733765 87.10831)
 		(end 196.042075 86.8)
@@
 			)
 		)
+	)
+	(zone
+		(net 47)
+		(net_name "+3V3")
+		(layer "In2.Cu")
+		(hatch edge 0.5)
+		(connect_pads
+			(clearance 0)
+		)
+		(min_thickness 0.25)
+		(filled_areas_thickness no)
+		(fill yes
+			(thermal_gap 0.5)
+			(thermal_bridge_width 0.5)
+		)
+		(polygon
+			(pts
+				(xy 207 71.5) (xy 210.2 71.5) (xy 210.2 68.8) (xy 214.2 68.8) (xy 214.2 66) (xy 207 66)
+			)
+		)

Commit message: linea de transmision ruteada
Parts:
- moved AE1 2.35 mm to (188.0, 62.0)
- moved J3 1.08 mm to (218.3, 84.4)
- moved J5 0.47 mm to (217.7, 75.1)
Routing:
- net Net-(U5-RF_IN): track 7.78 -> 0.02 mm
- net GND: track 128.2 -> 132.3 mm, vias 35 -> 71
- net /USB_D-: track 8.80 -> 9.88 mm
- net /USB_D+: track 8.80 -> 9.88 mm
- net VBUS: track 19.9 -> 21.0 mm
- added copper zone on F.Cu, net Net-(U5-RF_IN)

Commit message: Update flight_comp_srad-2026.kicad_pcb
1ra versión serigrafía
Parts:
- moved G*** 0.61 mm to (197.7, 69.6)
- renumbered U6 to FLASH
Other:
- board text added: "ADXL ACCL."
- board text added: "FLASH"
- board text added: "IIM-20670 ACCL & GYRO"
- board text added: "LED1"
- board text added: "LED2"
- board text added: "MAX M10M GPS"
- board text added: "MS5611 BAROM."
- board text added: "Pensa Piccolo, Vito Pérez Losada, Javier Baltasar Stefoni Rey Iraola, Pedro"
- board text added: "SWITCH 1"
- board text added: "SWITCH 2"
Changed lines of the file:
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@@
 	(footprint "my_lib:Logo_ITBA_rocketry"
 		(layer "F.Cu")
-		(at 197.641396 68.971604)
+		(at 197.741396 69.571604)
 		(property "Reference" "G***"
 			(at 0.5 -7.5 0)
@@
 			(at 0 -3.45 0)
 			(layer "F.SilkS")
+			(hide yes)
 			(effects
 				(font
@@
 			(at -7.9175 4.815 90)
 			(layer "F.SilkS")
+			(hide yes)
 			(effects
 				(font
@@
 			(at 2 0 0)
 			(layer "F.SilkS")
+			(hide yes)
 			(effects
 				(font
@@
 			(at 2.415 1.4 180)
 			(layer "F.SilkS")
+			(hide yes)
 			(effects
 				(font
@@
 		(tags "LED")
 		(property "Reference" "D2"
-			(at 2 0 180)
+			(at 2.1875 0 180)
 			(layer "F.SilkS")
+			(hide yes)
 			(effects
 				(font
@@
 			(at 1.925 -3.365 90)
 			(layer "F.SilkS")
+			(hide yes)
 			(effects
 				(font
@@
 			(at -13.65556 9.3391 90)
 			(layer "F.SilkS")
+			(hide yes)
 			(effects
 				(font
@@
 		(descr "SOIC, 8 Pin (JEITA/EIAJ 08-001-BBA and Atmel/Microchip, 208 mils width, https://www.jeita.or.jp/japanese/standard/book/ED-7311-19/#target/page_no=21, https://ww1.microchip.com/downloads/en/DeviceDoc/20005045C.pdf#page=23, https://ww1.microchip.com/downloads/en/DeviceDoc/doc2535.pdf#page=162), generated with kicad-footprint-generator ipc_gullwing_generator.py")
 		(tags "SOIC SO P-SOP SOP SOP-8 SO SO-8 8S2 S2AE/F K04-056 CASE-751BE SO8W 8-Pin-SOIC PSA W8-2 W8-4 W8MS-1")
-		(property "Reference" "U6"
-			(at -4.9175 -3.78 90)
+		(property "Reference" "FLASH"
+			(at 0.87 -20.13 270)
 			(layer "F.SilkS")
+			(hide yes)
 			(effects
 				(font
@@
 			(layer "F.Fab")
 		)
-		(fp_text user "${REFERENCE}"
+		(fp_text user "U6"
 			(at 0 0 90)
 			(layer "F.Fab")
@@
 			(at 0 1.65 90)
 			(layer "B.SilkS")
+			(hide yes)
 			(effects
 				(font
@@
 			(at 4.285 -3.27 90)
 			(layer "B.SilkS")
+			(hide yes)
 			(effects
 				(font
@@
 			(at 0 1.43 0)
 			(layer "B.SilkS")
+			(hide yes)
 			(effects
 				(font
@@
 			(at 0 1.43 0)
 			(layer "B.SilkS")
+			(hide yes)
 			(effects
 				(font
@@
 		(layer "Edge.Cuts")
 	)
+	(gr_text "Pensa Piccolo, Vito\nPérez Losada, Javier Baltasar\nStefoni Rey Iraola, Pedro"
+		(at 157.5 65.8 0)
+		(layer "F.SilkS")
+		(effects
+			(font
+				(size 1 1)
+				(thickness 0.2)
+				(bold yes)
+			)
+			(justify left bottom)
+		)
+	)
+	(gr_text "SWITCH 1"
+		(at 214.4 67.8 0)
+		(layer "F.SilkS")
+		(effects
+			(font
+				(size 0.7 0.7)
+				(thickness 0.175)
+				(bold yes)
+			)
+			(justify left bottom)
+		)
+	)
+	(gr_text "FLASH\n"
+		(at 212.5 77.3 270)
+		(layer "F.SilkS")
+		(effects
+			(font
+				(size 1 1)
+				(thickness 0.2)
+				(bold yes)
+			)
+			(justify left bottom)
+		)
+	)
+	(gr_text "MAX M10M\nGPS"
+		(at 173.5 72.6 0)
+		(layer "F.SilkS")
+		(effects
+			(font
+				(size 0.7 0.7)
+				(thickness 0.175)
+				(bold yes)
+			)
+			(justify right bottom)
+		)
+	)
+	(gr_text "LED2"
+		(at 203.2 96.5 270)
+		(layer "F.SilkS")
+		(effects
+			(font
+				(size 0.5 0.5)
+				(thickness 0.125)
+				(bold yes)
+			)
+			(justify left bottom)
+		)
+	)
+	(gr_text "SWITCH 2"
+		(at 191.5 91.2 0)
+		(layer "F.SilkS")
+		(effects
+			(font
+				(size 0.5 0.5)
+				(thickness 0.125)
+				(bold yes)
+			)
+			(justify left bottom)
+		)
+	)
+	(gr_text "LED1\n"
+		(at 199.3 97.2 90)
+		(layer "F.SilkS")
+		(effects
+			(font
+				(size 0.5 0.5)
+				(thickness 0.125)
+				(bold yes)
+			)
+			(justify left bottom)
+		)
+	)
+	(gr_text "ADXL ACCL."
+		(at 210.5 63.5 0)
+		(layer "B.SilkS")
+		(effects
+			(font
+				(size 0.7 0.7)
+				(thickness 0.175)
+				(bold yes)
+			)
+			(justify left bottom mirror)
+		)
+	)
+	(gr_text "MS5611 \nBAROM.\n"
+		(at 205.6 76.9 270)
+		(layer "B.SilkS")
+		(effects
+			(font
+				(size 0.7 0.7)
+				(thickness 0.175)
+				(bold yes)
+			)
+			(justify left bottom mirror)
+		)
+	)
+	(gr_text "IIM-20670\nACCL & GYRO\n"
+		(at 193.2 71.5 0)
+		(layer "B.SilkS")
+		(effects
+			(font
+				(size 0.7 0.7)
+				(thickness 0.175)
+				(bold yes)
+			)
+			(justify left bottom mirror)
+		)
+	)
 	(segment

Commit message: Cambio de regulador de tensión - chequear impedancia de línea
Parts:
- removed H2, H3, H4: MountingHole, MountingHole:MountingHole_2.5mm
- removed U2: NCP1117-3.3_SOT223, Package_TO_SOT_SMD:SOT-223-3_TabPin2
- added H5: MountingHole, MountingHole:MountingHole_3mm, F.Cu at (163.0, 85.4)
- added H6: MountingHole, MountingHole:MountingHole_3mm, F.Cu at (153.9, 63.2)
- added H7: MountingHole, MountingHole:MountingHole_3mm, F.Cu at (218.2, 63.3)
- added H8: MountingHole, MountingHole:MountingHole_3mm, F.Cu at (218.6, 98.1)
- added U8: TPS73733DCQ, Package_TO_SOT_SMD:SOT-223-6, F.Cu at (209.0, 96.1)
- H1: footprint MountingHole:MountingHole_2.5mm -> MountingHole:MountingHole_3mm
- moved H1 11.3 mm to (163.5, 69.2)
- moved G*** 1.84 mm to (199.1, 68.4)
- renumbered FLASH to U6
Connections:
- net Net-(U5-RF_IN) renamed /RF_IN
Routing:
- net +3V3: track 145.4 -> 149.3 mm, vias 32 -> 27
- net GND: track 132.3 -> 134.5 mm
- net VBUS: track 21.0 -> 20.2 mm, vias 2 -> 6
Other:
- board text added: "SRAD Flight Computer 2026"
